Commit message: stable

File: urdf/aerial_arm_ndt.xacro (robot description, xacro)
@@ -16,6 +16,6 @@
   <parent link="base_link"/>
   <child link="orientation_link"/>
-  <origin rpy="${pi/2} 0 -${pi/2}" xyz="0.0 0 0.0"/>
-  <!-- <origin rpy="${pi} 0 -${pi/2}" xyz="0.15 0 -0.07"/> -->
+  <!-- <origin rpy="${pi/2} 0 -${pi/2}" xyz="0.0 0 0.0"/> -->
+  <origin rpy="${pi} 0 -${pi/2}" xyz="0.15 0 -0.07"/>
 </joint>
 <link name="orientation_link"/>
@@ -180,6 +180,6 @@
   <axis xyz="0.0 1.0 -0.0"/>
   <limit
-      lower="-0.785375"
-      upper="0.785375"
+      lower="-3.1415"
+      upper="3.1415"
       effort="5"
       velocity="1.57"

File: urdf/aerial_arm_posctl.xacro (robot description, xacro)
@@ -2,5 +2,5 @@
 <robot name="aerial_arm" xmlns:xacro="http://www.ros.org/wiki/xacro">
 <xacro:include filename="$(find arm_description)/urdf/materials.xacro" />
-<xacro:include filename="$(find arm_description)/urdf/aerial_arm.trans" />
+<xacro:include filename="$(find arm_description)/urdf/aerial_arm_posctl.trans" />
 <xacro:include filename="$(find arm_description)/urdf/aerial_arm.gazebo" />
 	<xacro:property name="fric" value="0.005" />

File: urdf/mod/aerial_arm_cam.xacro (robot description, xacro)
@@ -17,5 +17,4 @@
   <child link="orientation_link"/>
   <origin rpy="${pi/2} 0 -${pi/2}" xyz="0.0 0 0.0"/>
-  <!-- <origin rpy="${pi} 0 -${pi/2}" xyz="0.15 0 -0.07"/> -->
 </joint>
 <link name="orientation_link"/>
@@ -276,4 +275,68 @@
 	</sensor>
 </gazebo>
+  <!-- CAMERA SENSOR -->
+   <link name="camera2_link">
+    <inertial>
+      <origin rpy="0 0 0" xyz="0 0 0"/>
+      <mass value="0.01"/>
+      <xacro:insert_block name="arm_inertia" />
+    </inertial>
+    <visual>
+      <origin rpy="0 0 0" xyz="0.0 0.0 0"/>
+      <geometry>
+        <box size="0.01 0.01 0.01"/>
+      </geometry>
+	 <material name="red">
+	  <color rgba="${204/255} ${0/255} ${0/255} 1.0"/>
+	</material>
+    </visual>
+    <collision>
+      <origin rpy="0 0 0" xyz="0.0 0.0 0"/>
+      <geometry>
+        <box size="0.02 0.02 0.02"/>
+      </geometry>
+    </collision>
+  </link>
+   <joint name="camera2_joint" type="fixed">
+    <origin rpy="0 1.57 1.57" xyz="0.012 0.025 0.0"/>
+    <parent link="Pitch_1"/>
+    <child link="camera2_link"/>
+  </joint>
+  <gazebo reference="camera2_link">
+    <sensor type="camera" name="camera2">
+      <update_rate>30.0</update_rate>
+      <camera name="head">
+        <horizontal_fov>1.3962634</horizontal_fov>
+        <image>
+          <width>800</width>
+          <height>600</height>
+          <format>R8G8B8</format>
+        </image>
+        <clip>
+          <near>0.02</near>
+          <far>300</far>
+        </clip>
+        <noise>
+          <type>gaussian</type>
+          <mean>0.0</mean>
+          <stddev>0.007</stddev>
+        </noise>
+      </camera>
+      <plugin name="camera_controller" filename="libgazebo_ros_camera.so">
+        <alwaysOn>true</alwaysOn>
+        <updateRate>0.0</updateRate>
+        <cameraName>/camera2</cameraName>
+        <imageTopicName>image_raw</imageTopicName>
+        <cameraInfoTopicName>camera_info</cameraInfoTopicName>
+        <frameName>camera_link</frameName>
+        <hackBaseline>0.07</hackBaseline>
+        <distortionK1>0.0</distortionK1>
+        <distortionK2>0.0</distortionK2>
+        <distortionK3>0.0</distortionK3>
+        <distortionT1>0.0</distortionT1>
+        <distortionT2>0.0</distortionT2>
+      </plugin>
+    </sensor>
+  </gazebo>
 <!-- <joint name="$tag_joint" type="fixed">-->
 <!--      <origin xyz="0 0.0225 0.0165" rpy="0 0 1.57"/>-->

File: urdf/mod/aerial_arm_mod.xacro (robot description, xacro)
@@ -6,16 +6,15 @@
 	<xacro:property name="fric" value="0.005" />
 	<xacro:property name="fric_ee" value="0.005" />
-<!--<link name="world"/>-->
-<!--<joint name="orientation_joint" type="fixed">-->
-<!--  <parent link="world"/>-->
-<!--  <child link="orientation_link"/>-->
-<!--  <origin rpy="${pi/2} 0 -${pi/2}" xyz="0 0 -0.001"/>-->
-<!--</joint>-->
-<!--<link name="base_link"/>-->
+<link name="world"/>
+<joint name="fix_joint" type="fixed">
+  <parent link="world"/>
+  <child link="base_link"/>
+  <origin rpy="${pi} 0 0" xyz="0 0 -0.2"/>
+</joint>
+<link name="base_link"/>
 <joint name="orientation_joint" type="fixed">
   <parent link="base_link"/>
   <child link="orientation_link"/>
   <origin rpy="${pi/2} 0 -${pi/2}" xyz="0.0 0 0.0"/>
-  <!-- <origin rpy="${pi} 0 -${pi/2}" xyz="0.15 0 -0.07"/> -->
 </joint>
 <link name="orientation_link"/>
@@ -264,4 +263,68 @@
  <dynamics damping="0.0" friction="${fric_ee}"/>
 </joint>
+<!-- CAMERA SENSOR -->
+   <link name="camera_link">
+    <inertial>
+      <origin rpy="0 0 0" xyz="0 0 0"/>
+      <mass value="0.001"/>
+      <inertia ixx="1e-07" ixy="0.0" ixz="-0.0" iyy="1e-07" iyz="-0.0" izz="1e-07"/>
+    </inertial>
+    <visual>
+      <origin rpy="0 0 0" xyz="0.0 0.0 0"/>
+      <geometry>
+        <box size="0.01 0.01 0.01"/>
+      </geometry>
+	 <material name="red">
+	  <color rgba="${204/255} ${0/255} ${0/255} 1.0"/>
+	</material>
+    </visual>
+    <collision>
+      <origin rpy="0 0 0" xyz="0.0 0.0 0"/>
+      <geometry>
+        <box size="0.01 0.01 0.01"/>
+      </geometry>
+    </collision>
+  </link>
+   <joint name="camera_joint" type="fixed">
+    <origin rpy="0 ${pi/2} ${pi/2}" xyz="0.012 0.025 0.0"/>
+    <parent link="Pitch_1"/>
+    <child link="camera_link"/>
+  </joint>
+  <gazebo reference="camera_link">
+    <sensor type="camera" name="camera">
+      <update_rate>30.0</update_rate>
+      <camera name="head">
+        <horizontal_fov>1.3962634</horizontal_fov>
+        <image>
+          <width>800</width>
+          <height>600</height>
+          <format>R8G8B8</format>
+        </image>
+        <clip>
+          <near>0.02</near>
+          <far>300</far>
+        </clip>
+        <noise>
+          <type>gaussian</type>
+          <mean>0.0</mean>
+          <stddev>0.007</stddev>
+        </noise>
+      </camera>
+      <plugin name="camera_controller" filename="libgazebo_ros_camera.so">
+        <alwaysOn>true</alwaysOn>
+        <updateRate>0.0</updateRate>
+        <cameraName>/camera</cameraName>
+        <imageTopicName>image_raw</imageTopicName>
+        <cameraInfoTopicName>camera_info</cameraInfoTopicName>
+        <frameName>camera_link</frameName>
+        <hackBaseline>0.07</hackBaseline>
+        <distortionK1>0.0</distortionK1>
+        <distortionK2>0.0</distortionK2>
+        <distortionK3>0.0</distortionK3>
+        <distortionT1>0.0</distortionT1>
+        <distortionT2>0.0</distortionT2>
+      </plugin>
+    </sensor>
+  </gazebo>
 <gazebo reference="Roll_1">
 	<sensor name="contact_sensor" type="contact">
@@ -276,4 +339,8 @@
 	</sensor>
 </gazebo>
+  <gazebo>
+    <plugin name="gazebo_ros_control" filename="libgazebo_ros_control.so">
+    </plugin>
+  </gazebo>
 <!-- <joint name="$tag_joint" type="fixed">-->
 <!--      <origin xyz="0 0.0225 0.0165" rpy="0 0 1.57"/>-->
